File: sb-cnc-shield.kicad_pcb (KiCad board)
At the start: 2 copper layers, 68.6 x 53.3 mm, 67 parts, among them P1 X, P2 Y, P3 Z, P4 A, P5 Conn_01x05, P6 I2C, P7 ES_SETUP, P8 12V-36V, SW1 RESET, U1 ARDUINO_UNO_SHIELD, U2 X, U3 Y, U4 Z, U5 A

Commit message: 3d models
Parts:
- JP1, JP10, JP11, JP12, JP13, JP14, JP15, JP16, JP17, JP18, JP19, JP2, JP20, JP21, JP22, JP23, JP24, JP25, JP26, JP27, JP28, JP29, JP3, JP30, JP31, JP32, JP33, JP34, JP35, JP36, JP37, JP38, JP39, JP4, JP5, JP6, JP7, JP8, JP9: footprint footprints:Pin_100mil_Header_Straight_1x02 -> sb-cnc-shield:Pin_100mil_Header_Straight_1x02
- P1, P2, P3, P4: footprint Pin_Headers:Pin_Header_Straight_2x04 -> sb-cnc-shield:Pin_Header_Straight_2x04
- P6: footprint Pin_Headers:Pin_Header_Straight_1x04 -> sb-cnc-shield:Pin_Header_Straight_1x04
Other:
- board text added: "JLCJLCJLCJLC"
